Commit message: Nav2 i Moveit implemented

File: sirius_description/robots/sirius.urdf.xacro (robot description, xacro)
@@ -5,13 +5,9 @@
   <xacro:arg name="elevation" default="0.0"/>
   <xacro:arg name="imu_frequency" default="200.0"/>
-  <xacro:arg name="gazebo_origin" default="[-9.396, 16.082]"/>
   <xacro:arg name="stereo_fps" default="30"/>
   <xacro:arg name="year" default=""/>
   <xacro:arg name="manipulator" default="none"/>
-  <!-- Set to 'true' to use real hardware interfaces instead of Gazebo simulation -->
-  <xacro:arg name="use_real_hardware" default="false"/>
-  <!-- Set to 'true' for the Unity simulation (unity_sim): ros2_control talks to Unity
-       over rosbridge topics through topic_based_ros2_control instead of gz_ros2_control -->
-  <xacro:arg name="unity_sim" default="false"/>
+  <!-- ros2_control parameters for gz_ros2_control (sirius_gazebo passes its controllers.yaml) -->
+  <xacro:arg name="gazebo_controllers" default=""/>
   <xacro:property name="calibration_path" value="$(arg calibration_path)" />
   <xacro:if value="${calibration_path != ''}">
@@ -21,5 +17,4 @@
   <xacro:property name="elevation" value="$(arg elevation)" />
   <xacro:property name="imu_frequency" value="$(arg imu_frequency)" />
-  <xacro:property name="gazebo_origin" value="${$(arg gazebo_origin)}" />
   <xacro:property name="stereo_fps" value="$(arg stereo_fps)" />
   <xacro:property name="year" value="$(arg year)" />
@@ -81,26 +76,9 @@
   <xacro:joint parent="platform" child="gnss" xyz="${mechanical['gnss_xyz']}" />
   <!-- ================================================================
-       Wheel drive system — switches between real hardware and Gazebo.
+       ros2_control hardware — Gazebo (gz_ros2_control)
        ================================================================ -->
-  <xacro:property name="use_real_hardware" value="$(arg use_real_hardware)"/>
-  <xacro:property name="unity_sim" value="$(arg unity_sim)"/>
   <ros2_control name="SiriusWheelSystem" type="system">
     <hardware>
-      <xacro:if value="${use_real_hardware}">
-        <!-- ODrive topic-bridge plugin (communicates via relaxing_middleware) -->
-        <plugin>sirius_hw_interfaces/SiriusWheelsHW</plugin>
-        <param name="driver_namespaces">
-          /wheels_left/motor0,/wheels_left/motor1,/wheels_right/motor0,/wheels_right/motor1
-        </param>
-      </xacro:if>
-      <xacro:if value="${not use_real_hardware and unity_sim}">
-        <plugin>topic_based_ros2_control/TopicBasedSystem</plugin>
-        <param name="joint_commands_topic">/sirius/wheel_commands</param>
-        <param name="joint_states_topic">/sirius/wheel_states</param>
-        <param name="trigger_joint_command_threshold">-1</param>
-      </xacro:if>
-      <xacro:if value="${not use_real_hardware and not unity_sim}">
-        <plugin>gz_ros2_control/GazeboSimSystem</plugin>
-      </xacro:if>
+      <plugin>gz_ros2_control/GazeboSimSystem</plugin>
     </hardware>
     <xacro:macro name="wheel_interface" params="name">
@@ -120,138 +98,34 @@
     <xacro:wheel_interface name="front_right" />
   </ros2_control>
-  <xacro:if value="${manipulator != 'none'}">
-    <xacro:include filename="$(find sirius_description)/urdf/sirius/manipulators/$(arg manipulator).urdf.xacro" />
+  <xacro:if value="${manipulator == '6DOF'}">
+    <xacro:include filename="$(find sirius_description)/urdf/sirius/manipulators/6DOF.urdf.xacro" />
     <xacro:joint parent="platform" child="root_link" xyz="${mechanical['suspension_separation_x']/2} 0 ${mechanical['suspension_z'] + 0.045}" rpy="0 0 0"/>
-    <!-- Manipulator ros2_control system — real or simulated -->
-    <xacro:if value="${manipulator == '5DOF'}">
-      <ros2_control name="SiriusManipSystem" type="system">
-        <hardware>
-          <xacro:if value="${use_real_hardware}">
-            <plugin>sirius_hw_interfaces/SiriusManipHW</plugin>
-            <param name="state_topic">/manip/joint_states</param>
-            <param name="command_topic">/manip/set_joint_states</param>
-          </xacro:if>
-          <xacro:if value="${not use_real_hardware and unity_sim}">
-            <plugin>topic_based_ros2_control/TopicBasedSystem</plugin>
-            <param name="joint_commands_topic">/sirius/manip_commands</param>
-            <param name="joint_states_topic">/sirius/manip_states</param>
-            <param name="trigger_joint_command_threshold">-1</param>
-          </xacro:if>
-          <xacro:if value="${not use_real_hardware and not unity_sim}">
-            <plugin>gz_ros2_control/GazeboSimSystem</plugin>
-          </xacro:if>
-        </hardware>
-        <joint name="waist">
-          <command_interface name="position"/>
-          <command_interface name="velocity"/>
-          <command_interface name="effort"/>
-          <state_interface name="position"><param name="initial_value">0.0</param></state_interface>
-          <state_interface name="velocity"/>
-          <state_interface name="effort"/>
-        </joint>
-        <joint name="shoulder">
-          <command_interface name="position"/>
-          <command_interface name="velocity"/>
-          <command_interface name="effort"/>
-          <state_interface name="position"><param name="initial_value">0.0</param></state_interface>
-          <state_interface name="velocity"/>
-          <state_interface name="effort"/>
-        </joint>
-        <joint name="elbow">
-          <command_interface name="position"/>
-          <command_interface name="velocity"/>
-          <command_interface name="effort"/>
-          <state_interface name="position"><param name="initial_value">0.0</param></state_interface>
-          <state_interface name="velocity"/>
-          <state_interface name="effort"/>
-        </joint>
-        <joint name="wrist_lift">
-          <command_interface name="position"/>
-          <command_interface name="velocity"/>
-          <command_interface name="effort"/>
-          <state_interface name="position"><param name="initial_value">0.0</param></state_interface>
-          <state_interface name="velocity"/>
-          <state_interface name="effort"/>
-        </joint>
-        <joint name="wrist_turn">
-          <command_interface name="position"/>
-          <command_interface name="velocity"/>
-          <command_interface name="effort"/>
-          <state_interface name="position"><param name="initial_value">0.0</param></state_interface>
-          <state_interface name="velocity"/>
-          <state_interface name="effort"/>
-        </joint>
-        <joint name="wrist_spin">
-          <command_interface name="position"/>
-          <command_interface name="velocity"/>
-          <command_interface name="effort"/>
-          <state_interface name="position"><param name="initial_value">0.0</param></state_interface>
-          <state_interface name="velocity"/>
-          <state_interface name="effort"/>
-        </joint>
-      </ros2_control>
-    </xacro:if>
-    <xacro:if value="${manipulator == '6DOF'}">
-      <ros2_control name="SiriusManipSystem" type="system">
-        <hardware>
-          <xacro:if value="${use_real_hardware}">
-            <plugin>sirius_hw_interfaces/SiriusManipHW</plugin>
-            <param name="state_topic">/manip/joint_states</param>
-            <param name="command_topic">/manip/set_joint_states</param>
-          </xacro:if>
-          <xacro:if value="${not use_real_hardware and unity_sim}">
-            <plugin>topic_based_ros2_control/TopicBasedSystem</plugin>
-            <param name="joint_commands_topic">/sirius/manip_commands</param>
-            <param name="joint_states_topic">/sirius/manip_states</param>
-            <param name="trigger_joint_command_threshold">-1</param>
-          </xacro:if>
-          <xacro:if value="${not use_real_hardware and not unity_sim}">
-            <plugin>gz_ros2_control/GazeboSimSystem</plugin>
-          </xacro:if>
-        </hardware>
-        <joint name="joint_1">
+    <ros2_control name="SiriusManipSystem" type="system">
+      <hardware>
+        <plugin>gz_ros2_control/GazeboSimSystem</plugin>
+      </hardware>
+      <xacro:macro name="arm_joint_interface" params="name">
+        <joint name="${name}">
           <command_interface name="position"/>
           <state_interface name="position"><param name="initial_value">0.0</param></state_interface>
           <state_interface name="velocity"/>
         </joint>
-        <joint name="joint_2">
-          <command_interface name="position"/>
-          <state_interface name="position"><param name="initial_value">0.0</param></state_interface>
-          <state_interface name="velocity"/>
-        </joint>
-        <joint name="joint_3">
-          <command_interface name="position"/>
-          <state_interface name="position"><param name="initial_value">0.0</param></state_interface>
-          <state_interface name="velocity"/>
-        </joint>
-        <joint name="joint_4">
-          <command_interface name="position"/>
-          <state_interface name="position"><param name="initial_value">0.0</param></state_interface>
-          <state_interface name="velocity"/>
-        </joint>
-        <joint name="joint_5">
-          <command_interface name="position"/>
-          <state_interface name="position"><param name="initial_value">0.0</param></state_interface>
-          <state_interface name="velocity"/>
-        </joint>
-        <joint name="joint_6">
-          <command_interface name="position"/>
-          <state_interface name="position"><param name="initial_value">0.0</param></state_interface>
-          <state_interface name="velocity"/>
-        </joint>
-      </ros2_control>
-    </xacro:if>
-  </xacro:if>
-  <!-- Unity simulation only: IMU frame and the camera frame name used by unity_rs_publisher -->
-  <xacro:if value="${unity_sim}">
-    <link name="imu_link"/>
-    <xacro:joint parent="platform" child="imu_link" xyz="0 0 0.1"/>
-    <link name="front_color_optical_frame"/>
-    <xacro:joint parent="front_rgb_camera_optical" child="front_color_optical_frame"/>
+      </xacro:macro>
+      <xacro:arm_joint_interface name="joint_1"/>
+      <xacro:arm_joint_interface name="joint_2"/>
+      <xacro:arm_joint_interface name="joint_3"/>
+      <xacro:arm_joint_interface name="joint_4"/>
+      <xacro:arm_joint_interface name="joint_5"/>
+      <xacro:arm_joint_interface name="joint_6"/>
+      <xacro:arm_joint_interface name="joint_gripper_left"/>
+      <xacro:arm_joint_interface name="joint_gripper_right"/>
+    </ros2_control>
   </xacro:if>
 <gazebo>
     <!-- Plugin kontrolera -->
     <plugin filename="gz_ros2_control-system" name="gz_ros2_control::GazeboSimROS2ControlPlugin">
-      <parameters>$(find sirius_description)/config/controllers.yaml</parameters>
+      <xacro:if value="${'$(arg gazebo_controllers)' != ''}">
+        <parameters>$(arg gazebo_controllers)</parameters>
+      </xacro:if>
     </plugin>
     <!-- Plugin Odometrii -->

File: sirius_description/urdf/hp_4310/hp_4310.urdf.xacro (robot description, xacro)
@@ -16,43 +16,4 @@
     </collision>
   </link>
-  <!-- <gazebo reference="${prefix}_camera">
-      <visual>
-        <xacro:element xacro:name="xacro:${material}" />
-      </visual>
-      <sensor type="camera" name="${prefix}_camera">
-      <update_rate>30.0</update_rate>
-      <camera name="${prefix}_camera">
-        <horizontal_fov>${78*pi/180}</horizontal_fov>
-        <image>
-          <width>1920</width>
-          <height>1080</height>
-          <format>R8G8B8</format>
-        </image>
-        <clip>
-          <near>0.02</near>
-          <far>300</far>
-        </clip>
-        <noise>
-          <type>gaussian</type>
-          <mean>0.0</mean>
-          <stddev>0.007</stddev>
-        </noise>
-      </camera>
-      <plugin name="camera_controller" filename="libgazebo_ros_camera.so">
-        <alwaysOn>true</alwaysOn>
-        <updateRate>0.0</updateRate>
-        <cameraName>/${prefix}_camera</cameraName>
-        <imageTopicName>image_raw</imageTopicName>
-        <cameraInfoTopicName>camera_info</cameraInfoTopicName>
-        <frameName>/${prefix}_camera</frameName>
-        <hackBaseline>0.0</hackBaseline>
-        <distortionK1>0.0</distortionK1>
-        <distortionK2>0.0</distortionK2>
-        <distortionK3>0.0</distortionK3>
-        <distortionT1>0.0</distortionT1>
-        <distortionT2>0.0</distortionT2>
-      </plugin>
-    </sensor>
-  </gazebo> -->
 </xacro:macro>
 </robot>

File: sirius_description/urdf/oak-d-w/oak-d-w.urdf.xacro (robot description, xacro)
@@ -1,5 +1,5 @@
 <?xml version="1.0"?>
 <robot xmlns:xacro="http://ros.org/wiki/xacro">
-<xacro:macro name="oak-d-w" params="prefix:=oak-d-w collisions:=${xacro.load_yaml('$(find sirius_description)/urdf/oak-d-w/collisions.yaml')} stereo_fps:=^|30 imu_frequency:=^|200 datum:=^ elevation:=^ year:=^ calibration:=${xacro.load_yaml('$(find sirius_calibration)/kalibr/camimu/inflated/camimu-camchain-imucam.yaml')} imu_calibration:=${xacro.load_yaml('$(find sirius_calibration)/kalibr/camimu/inflated/camimu-imu.yaml')}">
+<xacro:macro name="oak-d-w" params="prefix:=oak-d-w collisions:=${xacro.load_yaml('$(find sirius_description)/urdf/oak-d-w/collisions.yaml')} stereo_fps:=^|30 imu_frequency:=^|200 datum:=^ elevation:=^ year:=^ calibration:=${xacro.load_yaml('$(find sirius_description)/config/calibration/camimu-camchain-imucam.yaml')} imu_calibration:=${xacro.load_yaml('$(find sirius_description)/config/calibration/camimu-imu.yaml')}">
   <xacro:property name="optical_offset_x" value="-0.01" />
   <xacro:property name="baseline" value="${sqrt(calibration.cam1.T_cn_cnm1[0][3]**2 + calibration.cam1.T_cn_cnm1[1][3]**2 + calibration.cam1.T_cn_cnm1[2][3]**2)}"/>
@@ -109,5 +109,6 @@
     <sensor name="${prefix}_camera" type="rgbd_camera">
       <topic>${prefix}/camera</topic>
-      <gz_frame_id>${prefix}_camera</gz_frame_id>
+      <!-- Image/depth data use the optical convention (z forward) -->
+      <gz_frame_id>${prefix}_rgb_camera_optical</gz_frame_id>
       <pose>0 0 0 0 0 0</pose>
       <always_on>1</always_on>
@@ -234,11 +235,4 @@
         </z>
       </magnetometer>
-      <!-- <plugin filename="libgazebo_ros_magnetometer_sensor.so" name="magnetometer_plugin">
-        <ros>
-            <namespace>/${prefix}_camera/imu</namespace>
-            <remapping>~/out:=mag</remapping>
-        </ros>
-        <frame_name>${prefix}_camera_imu_link</frame_name>
-      </plugin> -->
     </sensor>
   </gazebo>

File: sirius_description/urdf/sirius/gnss.urdf.xacro (robot description, xacro)
@@ -3,5 +3,5 @@
      https://www.sparkfun.com/products/21801 -->
 <robot xmlns:xacro="http://wiki.ros.org/xacro">
-<xacro:macro name="gnss" params="prefix:='' material collisions:=${xacro.load_yaml('$(find sirius_description)/urdf/sirius/collisions.yaml')} datum:=^ elevation:=^ horizontal_cep:=1.0 vertical_cep:=1.5 rate:=20.0 gazebo_origin:=^">
+<xacro:macro name="gnss" params="prefix:='' material collisions:=${xacro.load_yaml('$(find sirius_description)/urdf/sirius/collisions.yaml')} datum:=^ elevation:=^ horizontal_cep:=1.0 vertical_cep:=1.5 rate:=20.0">
   <xacro:property name="_prefix" value="${prefix + '_' if prefix else ''}"/>
   <!-- sqrt(-1/(2*ln(0.5))) = 0.8493218002880191 -->
@@ -30,5 +30,5 @@
       <always_on>1</always_on>
       <update_rate>20</update_rate>
-      <topic>/${prefix}/gps/fix</topic>
+      <topic>/${_prefix}gps/fix</topic>
       <gz_frame_id>${prefix}gnss</gz_frame_id>
       <navsat>

File: sirius_description/urdf/sirius/manipulators/6DOF.urdf.xacro (robot description, xacro)
@@ -209,11 +209,22 @@
       <origin xyz="0 -0.0016 0.0552" rpy="0 0 0"/>
     </collision>
-  </link>
+    <inertial>
+      <origin xyz="0 0 0.0552"/>
+      <mass value="0.05"/>
+      <inertia ixx="3.5e-5" ixy="0" ixz="0" iyy="3.0e-5" iyz="0" izz="7.7e-6"/>
+    </inertial>
+  </link>
+  <!-- Jaw opening per side: 0 = jaws touching (closed), 0.0326 = fully open (65.2 mm gap).
+       The joint limits leave 2 mm of travel beyond that working range: in DART a jaw
+       pressed against an active limit (e.g. by gravity) gets stuck there. MoveIt keeps
+       to the working range (sirius_moveit_config/config/joint_limits.yaml).
+       Both jaws are driven independently (no <mimic>): gz_ros2_control's mimic loop
+       oscillates and drove the jaws into their limits. -->
   <joint name="joint_gripper_left" type="prismatic">
-    <origin xyz="0 -0.02 0.05" rpy="0 0 0"/>
+    <origin xyz="0 -0.0174 0.05" rpy="0 0 0"/>
     <parent link="tcp_connector"/>
     <child link="gripper_left"/>
     <axis xyz="0 -1 0"/>
-    <limit lower="0" upper="0.03" effort="1000.0" velocity="0.5"/>
+    <limit lower="-0.002" upper="0.0346" effort="100.0" velocity="0.1"/>
   </joint>
   <link name="gripper_right">
@@ -233,11 +244,16 @@
       <origin xyz="0 0.0016 0.0552" rpy="0 0 0"/>
     </collision>
+    <inertial>
+      <origin xyz="0 0 0.0552"/>
+      <mass value="0.05"/>
+      <inertia ixx="3.5e-5" ixy="0" ixz="0" iyy="3.0e-5" iyz="0" izz="7.7e-6"/>
+    </inertial>
   </link>
   <joint name="joint_gripper_right" type="prismatic">
-    <origin xyz="0 0.02 0.05" rpy="0 0 0"/>
+    <origin xyz="0 0.0174 0.05" rpy="0 0 0"/>
     <parent link="tcp_connector"/>
     <child link="gripper_right"/>
     <axis xyz="0 1 0"/>
-    <limit lower="0" upper="0.03" effort="1000.0" velocity="0.5"/>
+    <limit lower="-0.002" upper="0.0346" effort="100.0" velocity="0.1"/>
   </joint>
   <link name="tool"/>

File: sirius_description/urdf/sirius/wheel.urdf.xacro (robot description, xacro)
@@ -38,7 +38,4 @@
       <xacro:element xacro:name="xacro:${material}" />
     </visual>
-      <kd>5000.0</kd>
-      <kp>1e3</kp>
-      <max_vel>0.1</max_vel>
   </gazebo>
 </xacro:macro>
